File: CAD/esp-motioncontroller/DIFF_OUTPUT.kicad_sch (KiCad schematic)
At the start: 9 parts, among them U10 SP3485EN

Commit message: Feat: Allmost complete sepdriver
Parts:
- R26, R27: LCSC Part # C17477 -> C21189
- RN3: LCSC Part # (none) -> C29718
Connections:
- net ION: now also R26.2, R30.2; no longer R27.2, R30.1
- net IOP: now also R27.2, R30.1; no longer R26.2, R30.2
Changed lines of the file:
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@@
 	(hierarchical_label "IOP"
 		(shape input)
-		(at 187.96 86.36 0)
+		(at 187.96 93.98 0)
 		(effects
 			(font
@@
 	(hierarchical_label "ION"
 		(shape input)
-		(at 187.96 93.98 0)
+		(at 187.96 86.36 0)
 		(effects
 			(font
@@
 			)
 		)
-		(property "LCSC Part #" "C17477"
+		(property "LCSC Part #" "C21189"
 			(at 172.72 87.63 0)
 			(effects
@@
 			)
 		)
+		(property "LCSC Part #" "C29718"
+			(at 110.49 92.71 90)
+			(effects
+				(font
+					(size 1.27 1.27)
+				)
+				(hide yes)
+			)
+		)
 		(pin "1"
 		)
@@
 			)
 		)
-		(property "LCSC Part #" "C17477"
+		(property "LCSC Part #" "C21189"
 			(at 172.72 92.71 0)
 			(effects
