File: CAD/esp-motioncontroller/RS42-RS485.kicad_sch (KiCad schematic)
At the start: 9 parts, among them U2 SP3485EN

Commit message: Feat: Allmost complete sepdriver
Parts:
- R28, R29: LCSC Part # C17477 -> C21189
- RN1: LCSC Part # (none) -> C29718
Connections:
- net ION: now also R28.2, R31.2; no longer R29.2, R31.1
- net IOP: now also R29.2, R31.1; no longer R28.2, R31.2
Changed lines of the file:
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@@
 	(hierarchical_label "ION"
 		(shape input)
-		(at 170.18 91.44 0)
+		(at 170.18 83.82 0)
 		(effects
 			(font
@@
 	(hierarchical_label "IOP"
 		(shape input)
-		(at 170.18 83.82 0)
+		(at 170.18 91.44 0)
 		(effects
 			(font
@@
 			)
 		)
+		(property "LCSC Part #" "C29718"
+			(at 92.71 90.17 90)
+			(effects
+				(font
+					(size 1.27 1.27)
+				)
+				(hide yes)
+			)
+		)
 		(pin "1"
 		)
@@
 			)
 		)
-		(property "LCSC Part #" "C17477"
+		(property "LCSC Part #" "C21189"
 			(at 154.94 85.09 0)
 			(effects
@@
 			)
 		)
-		(property "LCSC Part #" "C17477"
+		(property "LCSC Part #" "C21189"
 			(at 154.94 90.17 0)
 			(effects
