File: CAD/esp-motioncontroller/esp-motioncontroller.kicad_pcb (KiCad board)
At the start: 2 copper layers, 99 x 77 mm, 70 parts, among them J1 Conn_01x06, J2 Screw_Terminal_01x08, J3 Screw_Terminal_01x08, J5 Screw_Terminal_01x03, J6 Screw_Terminal_01x08, J7 Screw_Terminal_01x03, U1 ESP32-S3-DevKitC, U11 LTV-817S, U12 LTV-817S, U13 LTV-817S, U14 LTV-817S, U15 AMS1117-3.3, U3 XL1509-5.0E1, U4 SP3485EN, U5 AM26LS31CDR, U6 LTV-817S, U7 LTV-817S, U8 LTV-817S, U9 LTV-817S, Y1 32.768khz 3215 12.5pf

Commit message: Feat: WIP Adding Differential input
Parts:
- moved H3 23.0 mm to (146.0, 141.0)
- moved H4 23.0 mm to (53.0, 141.0)
Routing:
- net GND: vias 265 -> 92
Other:
- board outline removed

Commit message: Feat: Additional driver
Parts:
- removed J5, J7: Screw_Terminal_01x03, TerminalBlock_Phoenix:TerminalBlock_Phoenix_PT-1,5-3-3.5-H_1x03_P3.50mm_Horizontal
- added C7: 0.1uF, Capacitor_SMD:C_0603_1608Metric, F.Cu at (73.6, 108.5)
- added C9: 0.1uF, Capacitor_SMD:C_0603_1608Metric, F.Cu at (134.0, 75.0)
- added J2: Screw_Terminal_01x10, TerminalBlock_Phoenix:TerminalBlock_Phoenix_PT-1,5-10-3.5-H_1x10_P3.50mm_Horizontal, F.Cu at (143.5, 122.5)
- added J4: Screw_Terminal_01x10, TerminalBlock_Phoenix:TerminalBlock_Phoenix_PT-1,5-10-3.5-H_1x10_P3.50mm_Horizontal, F.Cu at (59.5, 91.0)
- added J8: Screw_Terminal_01x10, TerminalBlock_Phoenix:TerminalBlock_Phoenix_PT-1,5-10-3.5-H_1x10_P3.50mm_Horizontal, F.Cu at (143.5, 84.0)
- added JP1: Jumper_2_Small_Open, TestPoint:TestPoint_2Pads_Pitch2.54mm_Drill0.8mm, F.Cu at (97.0, 121.5)
- added JP2: Jumper_2_Small_Open, TestPoint:TestPoint_2Pads_Pitch2.54mm_Drill0.8mm, F.Cu at (104.0, 122.0)
- added U10: AM26LS31CDR, Package_SO:SOIC-16_3.9x9.9mm_P1.27mm, F.Cu at (128.0, 71.0)
- added U2: AM26LV32EIDR, Package_SO:SOIC-16_3.9x9.9mm_P1.27mm, F.Cu at (69.0, 103.0)
- J2, J3, J6: value Screw_Terminal_01x08 -> Screw_Terminal_01x10; footprint TerminalBlock_Phoenix:TerminalBlock_Phoenix_PT-1,5-8-3.5-H_1x08_P3.50mm_Horizontal -> TerminalBlock_Phoenix:TerminalBlock_Phoenix_PT-1,5-10-3.5-H_1x10_P3.50mm_Horizontal
- moved D3 60.3 mm to (138.0, 110.0), turned to -90 degrees
- moved C5 55.9 mm to (133.5, 108.8), turned to -90 degrees
- moved C2 53.4 mm to (131.0, 108.8), turned to -90 degrees
- moved U3 50.6 mm to (127.0, 109.8), turned to -90 degrees
- moved J3 49.1 mm to (63.0, 136.5), turned to 0 degrees
- moved C3 46.7 mm to (118.0, 112.3), turned to 180 degrees
- moved R18 46.3 mm to (65.0, 131.0), turned to 180 degrees
- moved D1 43.8 mm to (122.5, 107.3), turned to -90 degrees
- moved L1 43.6 mm to (129.5, 99.8), turned to 90 degrees
- moved C6 43.5 mm to (118.0, 109.8), turned to 180 degrees
- moved J2 42.7 mm to (105.0, 136.5), turned to 0 degrees
- moved C8 40.4 mm to (118.0, 107.3), turned to 180 degrees
- moved R16 39.2 mm to (74.7, 131.0), turned to 180 degrees
- moved U6 38.2 mm to (67.5, 124.0), turned to 90 degrees
- moved C12 37.3 mm to (118.0, 104.8), turned to 180 degrees
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Connections:
- JP10 pad 1: GND_OPTO -> GND_OPTO_IN
- JP3 pad 1: GND_OPTO -> GND_OPTO_OUT
- JP4 pad 1: GND_OPTO -> GND_OPTO_OUT
- JP5 pad 1: GND_OPTO -> GND_OPTO_OUT
- JP6 pad 1: GND_OPTO -> GND_OPTO_IN
- JP7 pad 1: GND_OPTO -> GND_OPTO_IN
- JP8 pad 1: GND_OPTO -> GND_OPTO_OUT
- JP9 pad 1: GND_OPTO -> GND_OPTO_IN
- U1 pad 10: /InputOutput/ENBL_HO -> /esp32-s3/ENBL_HO
- U5 pad 4: /InputOutput/ENBL_HO -> /InputOutput/ENBL_HO_G1
Routing:
- net +3.3V: track 150.6 -> 94.3 mm, vias 2 -> 0
- net GND_OPTO: track 49.8 -> 0.00 mm
- net /InputOutput/OPTO_OUT_MCU_2: track 30.6 -> 0.00 mm
- net /InputOutput/OPTO_OUT_MCU_4: track 28.7 -> 0.00 mm
- net /InputOutput/OPTO_OUT_MCU_3: track 26.9 -> 0.00 mm
- net /InputOutput/OPTO_OUT_MCU_1: track 25.4 -> 0.00 mm
- net /InputOutput/RXD: track 25.1 -> 0.00 mm
- net Net-(J4-Pin_1): track 0.00 -> 23.1 mm
- net /InputOutput/TXD: track 22.6 -> 0.00 mm
- net /InputOutput/ENBL_HO: track 19.1 -> 0.00 mm
- net (no net): track 0.00 -> 19.1 mm
- net Net-(J4-Pin_2): track 0.00 -> 18.6 mm
- net /InputOutput/OPTO_IN_MCU_4: track 20.6 -> 2.14 mm
- net Net-(J4-Pin_8): track 0.00 -> 17.4 mm
- net Net-(J4-Pin_7): track 0.00 -> 16.2 mm
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Other:
- board outline added: 100 x 100 mm

Commit message: Feat: 485 single drivers
Parts:
- removed C1, C4: 20pf, Resistor_SMD:R_0603_1608Metric
- removed the J2 at (143.5, 122.5)
- removed Y1: 32.768khz 3215 12.5pf, Crystal:Crystal_SMD_3215-2Pin_3.2x1.5mm
- added C10: 0.1uF, Capacitor_SMD:C_0603_1608Metric, F.Cu at (230.5, -21.4)
- added C11: 0.1uF, Capacitor_SMD:C_0603_1608Metric, F.Cu at (231.8, 44.9)
- added C13: 0.1uF, Capacitor_SMD:C_0603_1608Metric, F.Cu at (160.8, 30.0)
- added C14: 0.1uF, Capacitor_SMD:C_0603_1608Metric, F.Cu at (199.3, 106.0)
- added C15: 0.1uF, Capacitor_SMD:C_0603_1608Metric, F.Cu at (199.0, 75.8)
- added C16: 0.1uF, Capacitor_SMD:C_0603_1608Metric, F.Cu at (230.5, -38.2)
- added C17: 0.1uF, Capacitor_SMD:C_0603_1608Metric, F.Cu at (231.8, -0.25)
- added C20: 0.1uF, Capacitor_SMD:C_0603_1608Metric, F.Cu at (229.5, -58.5)
- added C23: 0.1uF, Capacitor_SMD:C_0603_1608Metric, F.Cu at (231.8, 16.6)
- added J7: Screw_Terminal_01x10, TerminalBlock_Phoenix:TerminalBlock_Phoenix_PT-1,5-10-3.5-H_1x10_P3.50mm_Horizontal, F.Cu at (143.5, 122.5)
- added JP11: SolderJumper_3_Bridged12, Jumper:SolderJumper-3_P1.3mm_Bridged12_Pad1.0x1.5mm, F.Cu at (252.8, 47.6)
- added JP12: SolderJumper_3_Bridged12, Jumper:SolderJumper-3_P1.3mm_Bridged12_Pad1.0x1.5mm, F.Cu at (260.3, 47.6)
- added JP13: SolderJumper_2_Bridged, Jumper:SolderJumper-2_P1.3mm_Bridged_RoundedPad1.0x1.5mm, F.Cu at (271.3, 44.1)
- added JP14: SolderJumper_3_Bridged12, Jumper:SolderJumper-3_P1.3mm_Bridged12_Pad1.0x1.5mm, F.Cu at (254.0, 78.9)
- added JP15: SolderJumper_3_Bridged12, Jumper:SolderJumper-3_P1.3mm_Bridged12_Pad1.0x1.5mm, F.Cu at (261.5, 78.9)
- added JP16: SolderJumper_2_Bridged, Jumper:SolderJumper-2_P1.3mm_Bridged_RoundedPad1.0x1.5mm, F.Cu at (272.5, 75.4)
- added JP17: SolderJumper_3_Bridged12, Jumper:SolderJumper-3_P1.3mm_Bridged12_Pad1.0x1.5mm, F.Cu at (215.5, -17.9)
- added JP18: SolderJumper_3_Bridged12, Jumper:SolderJumper-3_P1.3mm_Bridged12_Pad1.0x1.5mm, F.Cu at (223.0, -17.9)
- added JP19: SolderJumper_2_Bridged, Jumper:SolderJumper-2_P1.3mm_Bridged_RoundedPad1.0x1.5mm, F.Cu at (234.0, -21.4)
- added JP20: SolderJumper_3_Bridged12, Jumper:SolderJumper-3_P1.3mm_Bridged12_Pad1.0x1.5mm, F.Cu at (216.5, 48.4)
- added JP21: SolderJumper_3_Bridged12, Jumper:SolderJumper-3_P1.3mm_Bridged12_Pad1.0x1.5mm, F.Cu at (224.0, 48.4)
- added JP22: SolderJumper_2_Bridged, Jumper:SolderJumper-2_P1.3mm_Bridged_RoundedPad1.0x1.5mm, F.Cu at (235.0, 44.9)
- added JP23: SolderJumper_3_Bridged12, Jumper:SolderJumper-3_P1.3mm_Bridged12_Pad1.0x1.5mm, F.Cu at (145.5, 33.5)
- added JP24: SolderJumper_3_Bridged12, Jumper:SolderJumper-3_P1.3mm_Bridged12_Pad1.0x1.5mm, F.Cu at (153.0, 33.5)
- added JP25: SolderJumper_2_Bridged, Jumper:SolderJumper-2_P1.3mm_Bridged_RoundedPad1.0x1.5mm, F.Cu at (164.0, 30.0)
- added JP26: SolderJumper_3_Bridged12, Jumper:SolderJumper-3_P1.3mm_Bridged12_Pad1.0x1.5mm, F.Cu at (184.0, 109.5)
- added JP27: SolderJumper_3_Bridged12, Jumper:SolderJumper-3_P1.3mm_Bridged12_Pad1.0x1.5mm, F.Cu at (191.5, 109.5)
- added JP28: SolderJumper_2_Bridged, Jumper:SolderJumper-2_P1.3mm_Bridged_RoundedPad1.0x1.5mm, F.Cu at (202.5, 106.0)
- added JP29: SolderJumper_3_Bridged12, Jumper:SolderJumper-3_P1.3mm_Bridged12_Pad1.0x1.5mm, F.Cu at (183.7, 79.2)
- added JP30: SolderJumper_3_Bridged12, Jumper:SolderJumper-3_P1.3mm_Bridged12_Pad1.0x1.5mm, F.Cu at (191.2, 79.2)
- added JP31: SolderJumper_2_Bridged, Jumper:SolderJumper-2_P1.3mm_Bridged_RoundedPad1.0x1.5mm, F.Cu at (202.2, 75.8)
- added JP32: SolderJumper_3_Bridged12, Jumper:SolderJumper-3_P1.3mm_Bridged12_Pad1.0x1.5mm, F.Cu at (215.5, -34.7)
- added JP33: SolderJumper_3_Bridged12, Jumper:SolderJumper-3_P1.3mm_Bridged12_Pad1.0x1.5mm, F.Cu at (223.0, -34.7)
- added JP34: SolderJumper_2_Bridged, Jumper:SolderJumper-2_P1.3mm_Bridged_RoundedPad1.0x1.5mm, F.Cu at (234.0, -38.2)
- added JP35: SolderJumper_3_Bridged12, Jumper:SolderJumper-3_P1.3mm_Bridged12_Pad1.0x1.5mm, F.Cu at (216.7, 3.25)
- added JP36: SolderJumper_3_Bridged12, Jumper:SolderJumper-3_P1.3mm_Bridged12_Pad1.0x1.5mm, F.Cu at (224.3, 3.25)
- added JP37: SolderJumper_2_Bridged, Jumper:SolderJumper-2_P1.3mm_Bridged_RoundedPad1.0x1.5mm, F.Cu at (235.2, -0.25)
- added JP38: SolderJumper_3_Bridged12, Jumper:SolderJumper-3_P1.3mm_Bridged12_Pad1.0x1.5mm, F.Cu at (145.5, 25.0)
- added JP39: SolderJumper_3_Bridged12, Jumper:SolderJumper-3_P1.3mm_Bridged12_Pad1.0x1.5mm, F.Cu at (153.0, 25.0)
- added JP40: SolderJumper_2_Bridged, Jumper:SolderJumper-2_P1.3mm_Bridged_RoundedPad1.0x1.5mm, F.Cu at (164.0, 21.5)
- added JP41: SolderJumper_3_Bridged12, Jumper:SolderJumper-3_P1.3mm_Bridged12_Pad1.0x1.5mm, F.Cu at (214.5, -55.0)
- added JP42: SolderJumper_3_Bridged12, Jumper:SolderJumper-3_P1.3mm_Bridged12_Pad1.0x1.5mm, F.Cu at (222.0, -55.0)
- added JP43: SolderJumper_2_Bridged, Jumper:SolderJumper-2_P1.3mm_Bridged_RoundedPad1.0x1.5mm, F.Cu at (233.0, -58.5)
- added JP44: SolderJumper_3_Bridged12, Jumper:SolderJumper-3_P1.3mm_Bridged12_Pad1.0x1.5mm, F.Cu at (216.7, 20.1)
- added JP45: SolderJumper_3_Bridged12, Jumper:SolderJumper-3_P1.3mm_Bridged12_Pad1.0x1.5mm, F.Cu at (224.3, 20.1)
- added JP46: SolderJumper_2_Bridged, Jumper:SolderJumper-2_P1.3mm_Bridged_RoundedPad1.0x1.5mm, F.Cu at (235.2, 16.6)
- added R24: 0R, Resistor_SMD:R_0603_1608Metric, F.Cu at (272.5, 77.9)
- added R25: 120R, Resistor_SMD:R_0603_1608Metric, F.Cu at (275.0, 78.9)
- added R26: 0R, Resistor_SMD:R_0603_1608Metric, F.Cu at (234.0, -16.9)
- added R27: 0R, Resistor_SMD:R_0603_1608Metric, F.Cu at (234.0, -18.9)
- added R28: 0R, Resistor_SMD:R_0603_1608Metric, F.Cu at (271.3, 48.6)
- added R29: 0R, Resistor_SMD:R_0603_1608Metric, F.Cu at (271.3, 46.6)
- added R30: 120R, Resistor_SMD:R_0603_1608Metric, F.Cu at (236.5, -17.9)
- added R31: 120R, Resistor_SMD:R_0603_1608Metric, F.Cu at (273.8, 47.6)
- added R32: 0R, Resistor_SMD:R_0603_1608Metric, F.Cu at (235.0, 49.4)
- added R33: 0R, Resistor_SMD:R_0603_1608Metric, F.Cu at (235.0, 47.4)
- added R34: 120R, Resistor_SMD:R_0603_1608Metric, F.Cu at (237.5, 48.4)
- added R35: 0R, Resistor_SMD:R_0603_1608Metric, F.Cu at (164.0, 34.5)
- added R36: 0R, Resistor_SMD:R_0603_1608Metric, F.Cu at (164.0, 32.5)
- added R37: 120R, Resistor_SMD:R_0603_1608Metric, F.Cu at (166.5, 33.5)
- added R38: 0R, Resistor_SMD:R_0603_1608Metric, F.Cu at (202.5, 110.5)
- added R39: 0R, Resistor_SMD:R_0603_1608Metric, F.Cu at (202.5, 108.5)
- added R4: 0R, Resistor_SMD:R_0603_1608Metric, F.Cu at (272.5, 79.9)
- added R40: 120R, Resistor_SMD:R_0603_1608Metric, F.Cu at (205.0, 109.5)
- added R41: 0R, Resistor_SMD:R_0603_1608Metric, F.Cu at (202.2, 80.2)
- added R42: 0R, Resistor_SMD:R_0603_1608Metric, F.Cu at (202.2, 78.2)
- added R43: 120R, Resistor_SMD:R_0603_1608Metric, F.Cu at (204.7, 79.2)
- added R44: 0R, Resistor_SMD:R_0603_1608Metric, F.Cu at (234.0, -33.7)
- added R45: 0R, Resistor_SMD:R_0603_1608Metric, F.Cu at (234.0, -35.7)
- added R46: 120R, Resistor_SMD:R_0603_1608Metric, F.Cu at (236.5, -34.7)
- added R47: 0R, Resistor_SMD:R_0603_1608Metric, F.Cu at (235.3, 4.25)
- added R48: 0R, Resistor_SMD:R_0603_1608Metric, F.Cu at (235.3, 2.25)
- added R49: 120R, Resistor_SMD:R_0603_1608Metric, F.Cu at (237.8, 3.25)
- added R50: 0R, Resistor_SMD:R_0603_1608Metric, F.Cu at (164.0, 26.0)
- added R51: 0R, Resistor_SMD:R_0603_1608Metric, F.Cu at (164.0, 24.0)
- added R52: 120R, Resistor_SMD:R_0603_1608Metric, F.Cu at (166.5, 25.0)
- added R53: 0R, Resistor_SMD:R_0603_1608Metric, F.Cu at (233.0, -54.0)
- added R54: 0R, Resistor_SMD:R_0603_1608Metric, F.Cu at (233.0, -56.0)
- added R55: 120R, Resistor_SMD:R_0603_1608Metric, F.Cu at (235.5, -55.0)
- added R56: 0R, Resistor_SMD:R_0603_1608Metric, F.Cu at (235.3, 21.1)
- added R57: 0R, Resistor_SMD:R_0603_1608Metric, F.Cu at (235.3, 19.1)
- added R58: 120R, Resistor_SMD:R_0603_1608Metric, F.Cu at (237.8, 20.1)
- added RN1: R_Pack04, Resistor_SMD:R_Array_Convex_4x0603, F.Cu at (256.3, 47.6)
- added RN10: R_Pack04, Resistor_SMD:R_Array_Convex_4x0603, F.Cu at (149.0, 25.0)
- added RN11: R_Pack04, Resistor_SMD:R_Array_Convex_4x0603, F.Cu at (218.0, -55.0)
- added RN12: R_Pack04, Resistor_SMD:R_Array_Convex_4x0603, F.Cu at (220.3, 20.1)
- added RN2: R_Pack04, Resistor_SMD:R_Array_Convex_4x0603, F.Cu at (257.5, 78.9)
- added RN3: R_Pack04, Resistor_SMD:R_Array_Convex_4x0603, F.Cu at (219.0, -17.9)
- added RN4: R_Pack04, Resistor_SMD:R_Array_Convex_4x0603, F.Cu at (220.0, 48.4)
- added RN5: R_Pack04, Resistor_SMD:R_Array_Convex_4x0603, F.Cu at (149.0, 33.5)
- added RN6: R_Pack04, Resistor_SMD:R_Array_Convex_4x0603, F.Cu at (187.5, 109.5)
- added RN7: R_Pack04, Resistor_SMD:R_Array_Convex_4x0603, F.Cu at (187.2, 79.2)
- added RN8: R_Pack04, Resistor_SMD:R_Array_Convex_4x0603, F.Cu at (219.0, -34.7)
- added RN9: R_Pack04, Resistor_SMD:R_Array_Convex_4x0603, F.Cu at (220.3, 3.25)
- added U16: SP3485EN, Package_SO:SOIC-8_3.9x4.9mm_P1.27mm, F.Cu at (229.5, 48.4)
- added U17: SP3485EN, Package_SO:SOIC-8_3.9x4.9mm_P1.27mm, F.Cu at (158.5, 33.5)
- added U18: SP3485EN, Package_SO:SOIC-8_3.9x4.9mm_P1.27mm, F.Cu at (197.0, 109.5)
- added U19: SP3485EN, Package_SO:SOIC-8_3.9x4.9mm_P1.27mm, F.Cu at (196.7, 79.2)
- added U20: SP3485EN, Package_SO:SOIC-8_3.9x4.9mm_P1.27mm, F.Cu at (228.5, -34.7)
- added U21: SP3485EN, Package_SO:SOIC-8_3.9x4.9mm_P1.27mm, F.Cu at (229.7, 3.25)
- added U22: SP3485EN, Package_SO:SOIC-8_3.9x4.9mm_P1.27mm, F.Cu at (158.5, 25.0)
- added U23: SP3485EN, Package_SO:SOIC-8_3.9x4.9mm_P1.27mm, F.Cu at (227.5, -55.0)
- added U24: SP3485EN, Package_SO:SOIC-8_3.9x4.9mm_P1.27mm, F.Cu at (229.7, 20.1)
- U10, U5: value AM26LS31CDR -> SP3485EN; footprint Package_SO:SOIC-16_3.9x9.9mm_P1.27mm -> Package_SO:SOIC-8_3.9x4.9mm_P1.27mm
- U2: value AM26LV32EIDR -> SP3485EN; footprint Package_SO:SOIC-16_3.9x9.9mm_P1.27mm -> Package_SO:SOIC-8_3.9x4.9mm_P1.27mm
- moved C7 204.9 mm to (268.1, 44.1), turned to 180 degrees
- moved U2 204.4 mm to (265.8, 47.6), turned to 0 degrees
- moved U5 196.4 mm to (267.0, 78.9), turned to 0 degrees
- moved C9 135.3 mm to (269.3, 75.4), turned to 180 degrees
- moved U10 134.1 mm to (228.5, -17.9), turned to 0 degrees
- moved C19 104.4 mm to (160.5, 21.5), turned to 180 degrees
- moved R14 0.26 mm to (133.7, 89.7)
- moved R13 0.23 mm to (133.6, 86.2)
Connections:
- C19 pad 1: 5V -> Net-(JP40-A)
- C7 pad 1: +3.3V -> Net-(JP13-A)
- C9 pad 1: 5V -> Net-(JP16-A)
- D3 pad 2: Net-(D3-A) -> VDC
- J4 pad 1: Net-(J4-Pin_1) -> unconnected-(J4-Pin_1-Pad1)
- J4 pad 10: 5V -> unconnected-(J4-Pin_10-Pad10)
- J4 pad 2: Net-(J4-Pin_2) -> unconnected-(J4-Pin_2-Pad2)
- J4 pad 3: Net-(J4-Pin_3) -> unconnected-(J4-Pin_3-Pad3)
- J4 pad 4: Net-(J4-Pin_4) -> unconnected-(J4-Pin_4-Pad4)
- J4 pad 5: Net-(J4-Pin_5) -> unconnected-(J4-Pin_5-Pad5)
- J4 pad 6: Net-(J4-Pin_6) -> unconnected-(J4-Pin_6-Pad6)
- J4 pad 7: Net-(J4-Pin_7) -> unconnected-(J4-Pin_7-Pad7)
- J4 pad 8: Net-(J4-Pin_8) -> unconnected-(J4-Pin_8-Pad8)
- J4 pad 9: GND -> unconnected-(J4-Pin_9-Pad9)
- J6 pad 1: Net-(J6-Pin_1) -> unconnected-(J6-Pin_1-Pad1)
- J6 pad 10: 5V -> unconnected-(J6-Pin_10-Pad10)
- J6 pad 2: Net-(J6-Pin_2) -> unconnected-(J6-Pin_2-Pad2)
- J6 pad 3: Net-(J6-Pin_3) -> unconnected-(J6-Pin_3-Pad3)
- J6 pad 4: Net-(J6-Pin_4) -> unconnected-(J6-Pin_4-Pad4)
- J6 pad 5: Net-(J6-Pin_5) -> unconnected-(J6-Pin_5-Pad5)
- J6 pad 6: Net-(J6-Pin_6) -> unconnected-(J6-Pin_6-Pad6)
- J6 pad 7: Net-(J6-Pin_7) -> unconnected-(J6-Pin_7-Pad7)
- J6 pad 8: Net-(J6-Pin_8) -> unconnected-(J6-Pin_8-Pad8)
- J6 pad 9: GND -> unconnected-(J6-Pin_9-Pad9)
- J8 pad 1: Net-(J8-Pin_1) -> unconnected-(J8-Pin_1-Pad1)
- J8 pad 10: 5V -> unconnected-(J8-Pin_10-Pad10)
- J8 pad 2: Net-(J8-Pin_2) -> unconnected-(J8-Pin_2-Pad2)
- J8 pad 3: Net-(J8-Pin_3) -> unconnected-(J8-Pin_3-Pad3)
- J8 pad 4: Net-(J8-Pin_4) -> unconnected-(J8-Pin_4-Pad4)
- J8 pad 5: Net-(J8-Pin_5) -> unconnected-(J8-Pin_5-Pad5)
- J8 pad 6: Net-(J8-Pin_6) -> unconnected-(J8-Pin_6-Pad6)
- J8 pad 7: Net-(J8-Pin_7) -> unconnected-(J8-Pin_7-Pad7)
- J8 pad 8: Net-(J8-Pin_8) -> unconnected-(J8-Pin_8-Pad8)
- J8 pad 9: GND -> unconnected-(J8-Pin_9-Pad9)
- U1 pad 4: /InputOutput/HO4 -> /esp32-s3/HO4
- U1 pad 5: /InputOutput/HO3 -> /esp32-s3/HO3
- U1 pad 6: /InputOutput/HO2 -> /esp32-s3/HO2
- U1 pad 7: /InputOutput/HO1 -> /esp32-s3/HO1
- U1 pad 8: Net-(U1-GPIO15/ADC2_CH4/32K_P) -> unconnected-(U1-GPIO15/ADC2_CH4/32K_P-Pad8)
- U1 pad 9: Net-(U1-GPIO16/ADC2_CH5/32K_N) -> unconnected-(U1-GPIO16/ADC2_CH5/32K_N-Pad9)
- U10 pad 1: /InputOutput/HO6 -> /InputOutput/DIFF_OUTPUT1/RXD'
- U10 pad 2: Net-(J8-Pin_6) -> Net-(JP18-B)
- U10 pad 3: Net-(J8-Pin_5) -> Net-(JP18-A)
- U10 pad 4: /InputOutput/ENBL_HO_G2 -> /InputOutput/DIFF_OUTPUT1/TXD'
- U10 pad 5: Net-(J8-Pin_7) -> GND
- U10 pad 6: Net-(J8-Pin_8) -> Net-(U10-A)
- U10 pad 7: /InputOutput/HO5 -> Net-(U10-B)
- U10 pad 8: GND -> Net-(JP19-A)
- U2 pad 1: Net-(J4-Pin_2) -> /InputOutput/DIFF_INPUT2/RXD'
- U2 pad 2: Net-(J4-Pin_1) -> Net-(JP12-A)
- U2 pad 3: /InputOutput/HI1 -> Net-(JP12-B)
- U2 pad 4: /InputOutput/ENBL_HI -> /InputOutput/DIFF_INPUT2/TXD'
- U2 pad 5: /InputOutput/HI1 -> GND
- U2 pad 6: Net-(J4-Pin_3) -> Net-(U2-A)
- U2 pad 7: Net-(J4-Pin_4) -> Net-(U2-B)
- U2 pad 8: GND -> Net-(JP13-A)
- U5 pad 1: /InputOutput/HO2 -> /InputOutput/DIFF_INPUT1/RXD'
- U5 pad 2: Net-(J6-Pin_6) -> Net-(JP15-A)
- U5 pad 3: Net-(J6-Pin_5) -> Net-(JP15-B)
- U5 pad 4: /InputOutput/ENBL_HO_G1 -> /InputOutput/DIFF_INPUT1/TXD'
- U5 pad 5: Net-(J6-Pin_7) -> GND
- U5 pad 6: Net-(J6-Pin_8) -> Net-(U5-A)
- U5 pad 7: /InputOutput/HO1 -> Net-(U5-B)
- U5 pad 8: GND -> Net-(JP16-A)
Routing:
- net +3.3V: track 94.3 -> 117.9 mm, vias 0 -> 12
- net Net-(J4-Pin_1): track 23.1 -> 0.00 mm
- net Net-(J6-Pin_2): track 22.9 -> 0.00 mm
- net Net-(J6-Pin_1): track 19.4 -> 0.00 mm
- net /InputOutput/HO2: track 19.3 -> 0.00 mm
- net (no net): track 19.1 -> 0.00 mm
- net Net-(J4-Pin_2): track 18.6 -> 0.00 mm
- net /InputOutput/HO3: track 18.5 -> 0.00 mm
- net Net-(J6-Pin_8): track 18.4 -> 0.00 mm
- net Net-(J4-Pin_8): track 17.4 -> 0.00 mm
- net Net-(J6-Pin_7): track 17.3 -> 0.00 mm
- net Net-(J4-Pin_7): track 16.2 -> 0.00 mm
- net 5V: track 114.8 -> 98.6 mm
- net Net-(J6-Pin_5): track 15.0 -> 0.00 mm
- net Net-(J6-Pin_3): track 14.2 -> 0.00 mm
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