File: CAD/esp-motioncontroller/esp-motioncontroller.kicad_pcb (KiCad board)
At the start: 2 copper layers, 100 x 100 mm, 77 parts, among them J1 Conn_01x06, J2 Screw_Terminal_01x10, J3 Screw_Terminal_01x10, J4 Screw_Terminal_01x10, J6 Screw_Terminal_01x10, J8 Screw_Terminal_01x10, U1 ESP32-S3-DevKitC, U10 AM26LS31CDR, U11 LTV-817S, U12 LTV-817S, U13 LTV-817S, U14 LTV-817S, U15 AMS1117-3.3, U2 AM26LV32EIDR, U3 XL1509-5.0E1, U4 SP3485EN, U5 AM26LS31CDR, U6 LTV-817S, U7 LTV-817S, U8 LTV-817S, U9 LTV-817S, Y1 32.768khz 3215 12.5pf

Commit message: Feat: Quaddrivers
Parts:
- removed C9: 0.1uF, Capacitor_SMD:C_0603_1608Metric
- removed the J2 at (143.5, 122.5)
- removed R14: 10k, Resistor_SMD:R_0603_1608Metric
- removed U10: AM26LS31CDR, Package_SO:SOIC-16_3.9x9.9mm_P1.27mm
- added J9: Screw_Terminal_01x10, TerminalBlock_Phoenix:TerminalBlock_Phoenix_PT-1,5-10-3.5-H_1x10_P3.50mm_Horizontal, F.Cu at (143.0, 84.0)
- added JP11: Jumper_2_Small_Open, TestPoint:TestPoint_2Pads_Pitch2.54mm_Drill0.8mm, F.Cu at (70.2, 85.6)
- added JP12: Jumper_2_Small_Open, TestPoint:TestPoint_2Pads_Pitch2.54mm_Drill0.8mm, F.Cu at (119.3, 73.4)
- added R4: 10k, Resistor_SMD:R_0603_1608Metric, F.Cu at (78.0, 91.0)
- moved R13 55.8 mm to (79.0, 75.0), turned to 90 degrees
- moved D1 54.4 mm to (131.5, 53.7)
- moved C3 54.0 mm to (121.1, 58.5), turned to 0 degrees
- moved D3 53.0 mm to (137.0, 57.0), turned to 90 degrees
- moved C6 49.0 mm to (121.1, 61.0), turned to 0 degrees
- moved L1 48.2 mm to (124.0, 52.0), turned to 180 degrees
- moved C2 47.8 mm to (131.0, 61.0)
- moved C5 47.8 mm to (133.5, 61.0)
- moved U3 47.8 mm to (127.0, 62.0)
- moved C8 44.0 mm to (121.1, 63.5), turned to 0 degrees
- moved C12 39.0 mm to (121.1, 66.0), turned to 0 degrees
- moved J8 38.5 mm to (143.0, 122.5)
- moved C21 35.5 mm to (134.2, 71.1), turned to -90 degrees
- moved D2 30.4 mm to (120.0, 69.0), turned to 180 degrees
- moved U15 26.7 mm to (128.0, 72.0), turned to 180 degrees
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Connections:
- net /InputOutput/A renamed /InputOutput/A_P
- net Net-(J4-Pin_1) renamed /InputOutput/HI1_P
- net Net-(J4-Pin_2) renamed /InputOutput/HI1_N
- net Net-(J4-Pin_3) renamed /InputOutput/HI2_P
- net Net-(J4-Pin_4) renamed /InputOutput/HI2_N
- net Net-(J4-Pin_5) renamed /InputOutput/HI3_P
- net Net-(J4-Pin_6) renamed /InputOutput/HI3_N
- net Net-(J4-Pin_7) renamed /InputOutput/HI4_P
- net Net-(J4-Pin_8) renamed /InputOutput/HI4_N
- net Net-(J6-Pin_3) renamed /InputOutput/HO2_P
- net Net-(J6-Pin_4) renamed /InputOutput/HO2_N
- net Net-(J6-Pin_7) renamed /InputOutput/HO4_N
- net Net-(J6-Pin_8) renamed /InputOutput/HO4_P
- C22 pad 1: +3.3V -> Net-(JP12-A)
- D3 pad 2: Net-(D3-A) -> VIN
- J6 pad 1: Net-(J6-Pin_1) -> /InputOutput/HO1_N
- J6 pad 2: Net-(J6-Pin_2) -> /InputOutput/HO1_P
- J6 pad 5: Net-(J6-Pin_5) -> /InputOutput/HO3_P
- J6 pad 6: Net-(J6-Pin_6) -> /InputOutput/HO3_N
- J8 pad 1: Net-(J8-Pin_1) -> unconnected-(J8-Pin_1-Pad1)
- J8 pad 2: Net-(J8-Pin_2) -> unconnected-(J8-Pin_2-Pad2)
- J8 pad 3: Net-(J8-Pin_3) -> unconnected-(J8-Pin_3-Pad3)
- J8 pad 4: Net-(J8-Pin_4) -> unconnected-(J8-Pin_4-Pad4)
- J8 pad 5: Net-(J8-Pin_5) -> unconnected-(J8-Pin_5-Pad5)
- J8 pad 6: Net-(J8-Pin_6) -> unconnected-(J8-Pin_6-Pad6)
- J8 pad 7: Net-(J8-Pin_7) -> unconnected-(J8-Pin_7-Pad7)
- J8 pad 8: Net-(J8-Pin_8) -> unconnected-(J8-Pin_8-Pad8)
- R11 pad 2: /InputOutput/B -> /InputOutput/B_N
- R12 pad 1: /InputOutput/B -> /InputOutput/B_N
- R13 pad 2: /InputOutput/B -> /InputOutput/ENBL_HO
- U1 pad 1: Net-(U1-3V3-Pad1) -> +3.3V
- U1 pad 10: /esp32-s3/ENBL_HO -> /InputOutput/ENBL_HO
- U1 pad 11: unconnected-(U1-GPIO18/ADC2_CH7-Pad11) -> /InputOutput/OPTO_IN_MCU_4
- U1 pad 12: unconnected-(U1-GPIO8/ADC1_CH7-Pad12) -> /InputOutput/OPTO_IN_MCU_3
- U1 pad 13: unconnected-(U1-GPIO3/ADC1_CH2-Pad13) -> /InputOutput/OPTO_IN_MCU_2
- U1 pad 15: /InputOutput/OPTO_IN_MCU_1 -> /InputOutput/ENBL_HI
- U1 pad 16: /InputOutput/OPTO_IN_MCU_2 -> /InputOutput/HI1
- U1 pad 17: /InputOutput/OPTO_IN_MCU_3 -> /InputOutput/HI2
- U1 pad 18: /InputOutput/OPTO_IN_MCU_4 -> /InputOutput/HI3
- U1 pad 19: unconnected-(U1-GPIO13/ADC2_CH2-Pad19) -> /InputOutput/HI4
- U1 pad 2: Net-(U1-3V3-Pad1) -> +3.3V
- U1 pad 20: unconnected-(U1-GPIO14/ADC2_CH3-Pad20) -> /InputOutput/OPTO_IN_MCU_1
- U1 pad 21: 5V -> Net-(JP11-A)
- U1 pad 27: unconnected-(U1-GPIO21-Pad27) -> /InputOutput/RE/DE
- U1 pad 30: /InputOutput/RE/DE -> unconnected-(U1-GPIO45-Pad30)
- U1 pad 32: /InputOutput/OPTO_OUT_MCU_1 -> unconnected-(U1-GPIO35-Pad32)
- U1 pad 33: /InputOutput/OPTO_OUT_MCU_2 -> unconnected-(U1-GPIO36-Pad33)
- U1 pad 34: /InputOutput/OPTO_OUT_MCU_3 -> unconnected-(U1-GPIO37-Pad34)
- U1 pad 35: /InputOutput/OPTO_OUT_MCU_4 -> unconnected-(U1-GPIO38-Pad35)
- U1 pad 36: unconnected-(U1-GPIO39/MTCK-Pad36) -> /InputOutput/OPTO_OUT_MCU_4
- U1 pad 37: unconnected-(U1-GPIO40/MTDO-Pad37) -> /InputOutput/OPTO_OUT_MCU_3
- U1 pad 38: unconnected-(U1-GPIO41/MTDI-Pad38) -> /InputOutput/OPTO_OUT_MCU_2
- U1 pad 39: unconnected-(U1-GPIO42/MTMS-Pad39) -> /InputOutput/OPTO_OUT_MCU_1
- U1 pad 4: /InputOutput/HO4 -> /InputOutput/HO1
- U1 pad 5: /InputOutput/HO3 -> /InputOutput/HO2
- U1 pad 6: /InputOutput/HO2 -> /InputOutput/HO3
- U1 pad 7: /InputOutput/HO1 -> /InputOutput/HO4
- U15 pad 2: +3.3V -> Net-(JP12-A)
- U2 pad 11: /InputOutput/HI1 -> /InputOutput/HI3
- U2 pad 12: unconnected-(U2-~{G}-Pad12) -> GND
- U2 pad 13: /InputOutput/HI1 -> /InputOutput/HI4
- U2 pad 5: /InputOutput/HI1 -> /InputOutput/HI2
- U5 pad 1: /InputOutput/HO2 -> /InputOutput/HO3
- U5 pad 10: Net-(J6-Pin_2) -> /InputOutput/HO1_N
- U5 pad 11: Net-(J6-Pin_1) -> /InputOutput/HO1_P
- U5 pad 15: /InputOutput/HO3 -> /InputOutput/HO2
- U5 pad 2: Net-(J6-Pin_6) -> /InputOutput/HO3_P
- U5 pad 3: Net-(J6-Pin_5) -> /InputOutput/HO3_N
- U5 pad 4: /InputOutput/ENBL_HO_G1 -> /InputOutput/ENBL_HO
- U5 pad 7: /InputOutput/HO1 -> /InputOutput/HO4
- U5 pad 9: /InputOutput/HO4 -> /InputOutput/HO1
Routing:
- net +VDC: track 13.4 -> 171.4 mm
- net +3.3V: track 94.3 -> 220.3 mm
- net 5V: track 114.8 -> 234.0 mm, vias 2 -> 0
- net /InputOutput/OPTO_OUT_MCU_4: track 0.00 -> 69.8 mm
- net /InputOutput/OPTO_OUT_MCU_3: track 0.00 -> 67.2 mm
- net /InputOutput/OPTO_OUT_MCU_2: track 0.00 -> 63.7 mm
- net /InputOutput/OPTO_OUT_MCU_1: track 0.00 -> 61.6 mm
- net /InputOutput/OPTO_IN_MCU_3: track 3.00 -> 51.7 mm
- net /InputOutput/OPTO_IN_MCU_4: track 2.14 -> 50.2 mm
- net /InputOutput/OPTO_IN_MCU_2: track 3.22 -> 49.6 mm
- net /InputOutput/ENBL_HI: track 0.00 -> 36.0 mm
- net Net-(JP11-A): track 0.00 -> 34.0 mm
- net GND_OPTO_OUT: track 0.00 -> 28.6 mm
- net /InputOutput/RXD: track 0.00 -> 28.3 mm
- net /InputOutput/OPTO_IN_MCU_1: track 0.00 -> 28.1 mm
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Other:
- outline, holes or cut-outs redrawn
- board text added: "5V"
- board text added: "A/P"
- board text added: "B/N"
- board text added: "ESP-Motion Rev 1.0.0"
- board text added: "GND"
- board text added: "VIN"

Commit message: Feat: Local libs, more devboards
Parts:
- removed J1: Conn_01x06, Connector_PinHeader_2.54mm:PinHeader_1x06_P2.54mm_Vertical
- added G***: LOGO, Library:LOGO, F.Cu at (126.0, 98.6)
- added kibuzzard-6890605B: G***, Library:kibuzzard-6890605B, F.Cu at (126.0, 86.1)
- C1, C4, R1, R10, R11, R12, R13, R15, R16, R17, R18, R19, R2, R20, R21, R22, R23, R3, R4, R5, R6, R7, R8, R9: footprint Resistor_SMD:R_0603_1608Metric -> Library:R_0603_1608Metric
- C12, C2, C21, C22, C3, C5, C6, C8: footprint Capacitor_SMD:C_1206_3216Metric -> Library:C_1206_3216Metric
- C18, C19, C7: footprint Capacitor_SMD:C_0603_1608Metric -> Library:C_0603_1608Metric
- D1, D2, D3: footprint Diode_SMD:D_SMA -> Library:D_SMA
- H1, H2, H3, H4: footprint MountingHole:MountingHole_3.2mm_M3_DIN965_Pad -> Library:MountingHole_3.2mm_M3_DIN965_Pad
- J2, J3, J4, J6, J8, J9: footprint TerminalBlock_Phoenix:TerminalBlock_Phoenix_PT-1,5-10-3.5-H_1x10_P3.50mm_Horizontal -> Library:TerminalBlock_Phoenix_PT-1,5-10-3.5-H_1x10_P3.50mm_Horizontal
- JP1, JP10, JP11, JP12, JP2, JP3, JP4, JP5, JP6, JP7, JP8, JP9: footprint TestPoint:TestPoint_2Pads_Pitch2.54mm_Drill0.8mm -> Library:TestPoint_2Pads_Pitch2.54mm_Drill0.8mm
- L1: footprint Inductor_SMD:L_SOREDE_SNR.1050_10x10x5mm -> Library:L_SOREDE_SNR.1050_10x10x5mm
- U1: footprint PCM_Espressif:ESP32-S3-DevKitC -> Library:ESP32-S3-DevKitC
- U11, U12, U13, U14, U6, U7, U8, U9: footprint Package_DIP:SMDIP-4_W9.53mm -> Library:SMDIP-4_W9.53mm
- U15: footprint Package_TO_SOT_SMD:SOT-223-3_TabPin2 -> Library:SOT-223-3_TabPin2
- U2, U5: footprint Package_SO:SOIC-16_3.9x9.9mm_P1.27mm -> Library:SOIC-16_3.9x9.9mm_P1.27mm
- U3, U4: footprint Package_SO:SOIC-8_3.9x4.9mm_P1.27mm -> Library:SOIC-8_3.9x4.9mm_P1.27mm
- Y1: footprint Crystal:Crystal_SMD_3215-2Pin_3.2x1.5mm -> Library:Crystal_SMD_3215-2Pin_3.2x1.5mm
Connections:
- J8 pad 1: unconnected-(J8-Pin_1-Pad1) -> GND
- J8 pad 2: unconnected-(J8-Pin_2-Pad2) -> GND
- J8 pad 3: unconnected-(J8-Pin_3-Pad3) -> GND
- J8 pad 4: unconnected-(J8-Pin_4-Pad4) -> GND
- J8 pad 5: unconnected-(J8-Pin_5-Pad5) -> GND
- J8 pad 6: unconnected-(J8-Pin_6-Pad6) -> GND
- J8 pad 7: unconnected-(J8-Pin_7-Pad7) -> GND
- J8 pad 8: unconnected-(J8-Pin_8-Pad8) -> GND
- U1 pad 42: /esp32-s3/rx -> unconnected-(U1-GPIO44/U0RXD-Pad42)
- U1 pad 43: /esp32-s3/tx -> unconnected-(U1-GPIO43/U0TXD-Pad43)
Routing:
- net /esp32-s3/tx: track 10.2 -> 0.00 mm
- net /esp32-s3/rx: track 9.25 -> 0.00 mm
- net /InputOutput/TXD: track 28.0 -> 30.7 mm
- net unconnected-(U1-GPIO48-Pad29): track 0.00 -> 2.54 mm
- net unconnected-(U1-GPIO47-Pad28): track 0.00 -> 2.54 mm
- net unconnected-(U1-GPIO45-Pad30): track 0.00 -> 2.54 mm
- net unconnected-(U1-GPIO44/U0RXD-Pad42): track 0.00 -> 2.54 mm
- net unconnected-(U1-GPIO43/U0TXD-Pad43): track 0.00 -> 2.54 mm
- net unconnected-(U1-GPIO38-Pad35): track 0.00 -> 2.54 mm
- net unconnected-(U1-GPIO37-Pad34): track 0.00 -> 2.54 mm
- net unconnected-(U1-GPIO36-Pad33): track 0.00 -> 2.54 mm
- net unconnected-(U1-GPIO35-Pad32): track 0.00 -> 2.54 mm
- net unconnected-(U1-GPIO20/USB_D+-Pad26): track 0.00 -> 2.54 mm
- net unconnected-(U1-GPIO19/USB_D--Pad25): track 0.00 -> 2.54 mm
- net unconnected-(U1-GPIO0-Pad31): track 0.00 -> 2.54 mm
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Other:
- board text added: "01N"
- board text added: "G1"
- board text added: "G2"
- board text added: "G3"
- board text added: "G4"
- board text added: "HIGHSPEED INPUTS"
- board text added: "HIGHSPEED OUTPUTS"
- board text added: "I1"
- board text added: "I1N"
- board text added: "I1P"
- board text added: "I2"
- board text added: "I2N"
- board text added: "I2P"
- board text added: "I3"
- board text added: "I3N"
- board text added: "I3P"
- board text added: "I4"
- board text added: "I4N"
- board text added: "I4P"
- board text added: "O1"
- board text added: "O1P"
- board text added: "O2"
- board text added: "O2N"
- board text added: "O2P"
- board text added: "O3"
- board text added: "O3N"
- board text added: "O3P"
- board text added: "O4"
- board text added: "O4N"
- board text added: "O4P"
- board text added: "OPTO-IN"
- board text added: "OPTO-OUT"
- board text added: "RS485"
- board text added: "Rev 1.0.0"
- board text added: "VDC"
- board text added: "VIN-7-40V"
- board text removed: "ESP-Motion Rev 1.0.0"
