File: CAD/esp-motioncontroller/esp-motioncontroller.kicad_sch (KiCad schematic)
At the start: 4 parts

Commit message: Feat: Quaddrivers
Other:
- sheet InputOutput ports: added ENBL_HI, ENBL_HO_G1, HI1, HI2, HI3, HI4; removed none
- sheet esp32-s3 ports: added ENBL_HI, HI1, HI2, HI3, HI4; removed none

Commit message: Feat: Local libs, more devboards
Parts:
- H1, H2, H3, H4: footprint MountingHole:MountingHole_3.2mm_M3_DIN965_Pad -> Library:MountingHole_3.2mm_M3_DIN965_Pad; symbol Mechanical:MountingHole_Pad -> Library:MountingHole_Pad
Changed lines of the file:
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@@
 	(generator_version "9.0")
 	(paper "A4")
+	(title_block
+		(date "2025-08-04")
+		(rev "1.0.0")
+	)
 	(wire
 		(pts
@@
 	)
 	(symbol
-		(lib_id "Mechanical:MountingHole_Pad")
+		(lib_id "Library:MountingHole_Pad")
 		(at 256.54 26.67 0)
 		(unit 1)
@@
 			)
 		)
-		(property "Footprint" "MountingHole:MountingHole_3.2mm_M3_DIN965_Pad"
+		(property "Footprint" "Library:MountingHole_3.2mm_M3_DIN965_Pad"
 			(at 256.54 26.67 0)
 			(effects
@@
 	)
 	(symbol
-		(lib_id "power:GND")
+		(lib_id "Library:GND")
 		(at 243.84 29.21 0)
 		(unit 1)
@@
 	)
 	(symbol
-		(lib_id "Mechanical:MountingHole_Pad")
+		(lib_id "Library:MountingHole_Pad")
 		(at 231.14 26.67 0)
 		(unit 1)
@@
 			)
 		)
-		(property "Footprint" "MountingHole:MountingHole_3.2mm_M3_DIN965_Pad"
+		(property "Footprint" "Library:MountingHole_3.2mm_M3_DIN965_Pad"
 			(at 231.14 26.67 0)
 			(effects
@@
 	)
 	(symbol
-		(lib_id "Mechanical:MountingHole_Pad")
+		(lib_id "Library:MountingHole_Pad")
 		(at 218.44 26.67 0)
 		(unit 1)
@@
 			)
 		)
-		(property "Footprint" "MountingHole:MountingHole_3.2mm_M3_DIN965_Pad"
+		(property "Footprint" "Library:MountingHole_3.2mm_M3_DIN965_Pad"
 			(at 218.44 26.67 0)
 			(effects
@@
 	)
 	(symbol
-		(lib_id "power:GND")
+		(lib_id "Library:GND")
 		(at 218.44 29.21 0)
 		(unit 1)
@@
 	)
 	(symbol
-		(lib_id "power:GND")
+		(lib_id "Library:GND")
 		(at 231.14 29.21 0)
 		(unit 1)
@@
 	)
 	(symbol
-		(lib_id "Mechanical:MountingHole_Pad")
+		(lib_id "Library:MountingHole_Pad")
 		(at 243.84 26.67 0)
 		(unit 1)
@@
 			)
 		)
-		(property "Footprint" "MountingHole:MountingHole_3.2mm_M3_DIN965_Pad"
+		(property "Footprint" "Library:MountingHole_3.2mm_M3_DIN965_Pad"
 			(at 243.84 26.67 0)
 			(effects
@@
 	)
 	(symbol
-		(lib_id "power:GND")
+		(lib_id "Library:GND")
 		(at 256.54 29.21 0)
 		(unit 1)
