File: CAD/esp-motioncontroller/esp32-s3.kicad_sch (KiCad schematic)
At the start: 20 parts, among them J1 Conn_01x06, J7 Screw_Terminal_01x03, U1 ESP32-S3-DevKitC, U15 AMS1117-3.3, U3 XL1509-5.0E1, Y1 32.768khz 3215 12.5pf

Commit message: Feat: Quaddrivers
Parts:
- removed J7: Screw_Terminal_01x03, TerminalBlock_Phoenix:TerminalBlock_Phoenix_PT-1,5-3-3.5-H_1x03_P3.50mm_Horizontal, symbol Connector:Screw_Terminal_01x03
- added JP11, JP12: Jumper_2_Small_Open, TestPoint:TestPoint_2Pads_Pitch2.54mm_Drill0.8mm, symbol Jumper:Jumper_2_Small_Open
- U1: now left out of the parts list
- U15: LCSC Part # SOT-223 -> C6186
Connections:
- net +3.3V: now also U1.1 (3V3), U1.2 (3V3), JP12.2 (B); no longer C22.1, U15.2 (VO)
- net 5V: now also JP11.2 (B); no longer U1.21 (5V)
- net HO1: now also U1.4 (GPIO4/ADC1_CH3); no longer U1.7 (GPIO7/ADC1_CH6)
- net HO2: now also U1.5 (GPIO5/ADC1_CH4); no longer U1.6 (GPIO6/ADC1_CH5)
- net HO3: now also U1.6 (GPIO6/ADC1_CH5); no longer U1.5 (GPIO5/ADC1_CH4)
- net HO4: now also U1.7 (GPIO7/ADC1_CH6); no longer U1.4 (GPIO4/ADC1_CH3)
- net OPTO_IN_MCU_1: now also U1.20 (GPIO14/ADC2_CH3); no longer U1.15 (GPIO9/ADC1_CH8)
- net OPTO_IN_MCU_2: now also U1.13 (GPIO3/ADC1_CH2); no longer U1.16 (GPIO10/ADC1_CH9)
- net OPTO_IN_MCU_3: now also U1.12 (GPIO8/ADC1_CH7); no longer U1.17 (GPIO11/ADC2_CH0)
- net OPTO_IN_MCU_4: now also U1.11 (GPIO18/ADC2_CH7); no longer U1.18 (GPIO12/ADC2_CH1)
- net OPTO_OUT_MCU_1: now also U1.39 (GPIO42/MTMS); no longer U1.32 (GPIO35)
- net OPTO_OUT_MCU_2: now also U1.38 (GPIO41/MTDI); no longer U1.33 (GPIO36)
- net OPTO_OUT_MCU_3: now also U1.37 (GPIO40/MTDO); no longer U1.34 (GPIO37)
- net OPTO_OUT_MCU_4: now also U1.36 (GPIO39/MTCK); no longer U1.35 (GPIO38)
- net RE/DE: now also U1.27 (GPIO21); no longer U1.30 (GPIO45)
- net HI4: now reaches U1.19 (GPIO13/ADC2_CH2)
- net VIN: now reaches D3.2 (A)
- new net: JP11.1 (A), U1.21 (5V)
- new net: C22.1, JP12.1 (A), U15.2 (VO)
- new net ENBL_HI: U1.15 (GPIO9/ADC1_CH8)
- new net HI1: U1.16 (GPIO10/ADC1_CH9)
- new net HI2: U1.17 (GPIO11/ADC2_CH0)
- new net HI3: U1.18 (GPIO12/ADC2_CH1)
Other:
- moved on the sheet: D3

Commit message: Feat: Local libs, more devboards
Parts:
- removed J1: Conn_01x06, Connector_PinHeader_2.54mm:PinHeader_1x06_P2.54mm_Vertical, symbol Connector_Generic:Conn_01x06
- C1, C4: footprint Resistor_SMD:R_0603_1608Metric -> Library:R_0603_1608Metric
- C12, C2, C21, C22, C3, C5, C6, C8: footprint Capacitor_SMD:C_1206_3216Metric -> Library:C_1206_3216Metric
- D1, D2, D3: footprint Diode_SMD:D_SMA -> Library:D_SMA
- JP11, JP12: footprint TestPoint:TestPoint_2Pads_Pitch2.54mm_Drill0.8mm -> Library:TestPoint_2Pads_Pitch2.54mm_Drill0.8mm; symbol Jumper:Jumper_2_Small_Open -> Library:Jumper_2_Small_Open
- L1: footprint Inductor_SMD:L_SOREDE_SNR.1050_10x10x5mm -> Library:L_SOREDE_SNR.1050_10x10x5mm; symbol Device:L -> Library:L
- U1: footprint PCM_Espressif:ESP32-S3-DevKitC -> Library:ESP32-S3-DevKitC; symbol PCM_Espressif:ESP32-S3-DevKitC -> Library:ESP32-S3-DevKitC
- U15: footprint Package_TO_SOT_SMD:SOT-223-3_TabPin2 -> Library:SOT-223-3_TabPin2; symbol Regulator_Linear:AMS1117-3.3 -> Library:AMS1117-3.3
- U3: footprint Package_SO:SOIC-8_3.9x4.9mm_P1.27mm -> Library:SOIC-8_3.9x4.9mm_P1.27mm; symbol Regulator_Switching:XL1509-5.0 -> Library:XL1509-5.0
- Y1: footprint Crystal:Crystal_SMD_3215-2Pin_3.2x1.5mm -> Library:Crystal_SMD_3215-2Pin_3.2x1.5mm
Connections:
- net rx: no longer names the net of U1.42 (GPIO44/U0RXD)
- net tx: no longer names the net of U1.43 (GPIO43/U0TXD)

Commit message: Feat: Fixed CI vendor prod files, and auto readme generation
Parts:
- C1, C4: LCSC (none) -> C1648; LCSC Part # C1648 -> (none)
- C12, C2, C21, C22, C3, C5, C6, C8: LCSC (none) -> C13585; LCSC Part # C13585 -> (none)
- D1, D2, D3: LCSC (none) -> C2480; LCSC Part # C2480 -> (none)
- L1: LCSC (none) -> C9187; LCSC Part # C9187 -> (none)
- U15: LCSC (none) -> C6186; LCSC Part # C6186 -> (none)
- U3: LCSC (none) -> C61063; LCSC Part # C61063 -> (none)
- Y1: LCSC (none) -> C32346; LCSC Part # C32346 -> (none)
Changed lines of the file:
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@@
-			)
-		)
-		(property "LCSC Part #" "C13585"
-			(at 266.7 78.74 0)
-			(effects
-				(font
-					(size 1.27 1.27)
-				)
-				(hide yes)
 			)
 		)
@@
 			)
 		)
+		(property "LCSC" "C13585"
+			(at 266.7 78.74 0)
+			(effects
+				(font
+					(size 1.27 1.27)
+				)
+				(hide yes)
+			)
+		)
 		(pin "1"
 		)
@@
 			)
 		)
-		(property "LCSC Part #" "C13585"
-			(at 254 78.74 0)
-			(effects
-				(font
-					(size 1.27 1.27)
-				)
-				(hide yes)
-			)
-		)
 		(property "TEST" ""
 			(at 254 78.74 0)
@@
 			)
 		)
+		(property "LCSC" "C13585"
+			(at 254 78.74 0)
+			(effects
+				(font
+					(size 1.27 1.27)
+				)
+				(hide yes)
+			)
+		)
 		(pin "1"
 		)
@@
 			)
 		)
-		(property "LCSC Part #" "C13585"
-			(at 193.04 78.74 0)
-			(effects
-				(font
-					(size 1.27 1.27)
-				)
-				(hide yes)
-			)
-		)
 		(property "TEST" ""
 			(at 193.04 78.74 0)
@@
 		)
 		(property "MPN" ""
+			(at 193.04 78.74 0)
+			(effects
+				(font
+					(size 1.27 1.27)
+				)
+				(hide yes)
+			)
+		)
+		(property "LCSC" "C13585"
 			(at 193.04 78.74 0)
 			(effects
@@
 			)
 		)
-		(property "LCSC Part #" "C1648"
-			(at 43.18 46.99 0)
-			(effects
-				(font
-					(size 1.27 1.27)
-				)
-				(hide yes)
-			)
-		)
 		(property "MPN" ""
 			(at 43.18 46.99 90)
@@
 			)
 		)
+		(property "LCSC" "C1648"
+			(at 43.18 46.99 90)
+			(effects
+				(font
+					(size 1.27 1.27)
+				)
+				(hide yes)
+			)
+		)
 		(pin "1"
 		)
@@
 			)
 		)
-		(property "LCSC Part #" "C13585"
-			(at 260.35 78.74 0)
-			(effects
-				(font
-					(size 1.27 1.27)
-				)
-				(hide yes)
-			)
-		)
 		(property "TEST" ""
 			(at 260.35 78.74 0)
@@
 		)
 		(property "MPN" ""
+			(at 260.35 78.74 0)
+			(effects
+				(font
+					(size 1.27 1.27)
+				)
+				(hide yes)
+			)
+		)
+		(property "LCSC" "C13585"
 			(at 260.35 78.74 0)
 			(effects
@@
 			)
 		)
-		(property "LCSC Part #" "C9187"
-			(at 237.49 74.93 0)
-			(effects
-				(font
-					(size 1.27 1.27)
-				)
-				(hide yes)
-			)
-		)
 		(property "MPN" ""
+			(at 237.49 74.93 90)
+			(effects
+				(font
+					(size 1.27 1.27)
+				)
+				(hide yes)
+			)
+		)
+		(property "LCSC" "C9187"
 			(at 237.49 74.93 90)
 			(effects
@@
 			)
 		)
-		(property "LCSC Part #" "C1648"
-			(at 43.18 39.37 0)
-			(effects
-				(font
-					(size 1.27 1.27)
-				)
-				(hide yes)
-			)
-		)
 		(property "MPN" ""
 			(at 43.18 39.37 90)
@@
 			)
 		)
+		(property "LCSC" "C1648"
+			(at 43.18 39.37 90)
+			(effects
+				(font
+					(size 1.27 1.27)
+				)
+				(hide yes)
+			)
+		)
 		(pin "1"
 		)
@@
 			)
 		)
-		(property "LCSC Part #" "C13585"
-			(at 205.74 31.75 0)
-			(effects
-				(font
-					(size 1.27 1.27)
-				)
-				(hide yes)
-			)
-		)
 		(property "TEST" ""
 			(at 205.74 31.75 0)
@@
 		)
 		(property "MPN" ""
+			(at 205.74 31.75 0)
+			(effects
+				(font
+					(size 1.27 1.27)
+				)
+				(hide yes)
+			)
+		)
+		(property "LCSC" "C13585"
 			(at 205.74 31.75 0)
 			(effects
@@
 			)
 		)
-		(property "LCSC Part #" "C13585"
-			(at 247.65 78.74 0)
-			(effects
-				(font
-					(size 1.27 1.27)
-				)
-				(hide yes)
-			)
-		)
 		(property "TEST" ""
 			(at 247.65 78.74 0)
@@
 		)
 		(property "MPN" ""
+			(at 247.65 78.74 0)
+			(effects
+				(font
+					(size 1.27 1.27)
+				)
+				(hide yes)
+			)
+		)
+		(property "LCSC" "C13585"
 			(at 247.65 78.74 0)
 			(effects
@@
 			)
 		)
-		(property "LCSC Part #" "C2480"
-			(at 227.33 78.74 0)
-			(effects
-				(font
-					(size 1.27 1.27)
-				)
-				(hide yes)
-			)
-		)
 		(property "MPN" ""
+			(at 227.33 78.74 90)
+			(effects
+				(font
+					(size 1.27 1.27)
+				)
+				(hide yes)
+			)
+		)
+		(property "LCSC" "C2480"
 			(at 227.33 78.74 90)
 			(effects
@@
 			)
 		)
-		(property "LCSC Part #" "C6186"
+		(property "MPN" ""
 			(at 227.33 27.94 0)
 			(effects
@@
 			)
 		)
-		(property "MPN" ""
+		(property "LCSC" "C6186"
 			(at 227.33 27.94 0)
 			(effects
@@
 			)
 		)
-		(property "LCSC Part #" "C13585"
-			(at 246.38 31.75 0)
-			(effects
-				(font
-					(size 1.27 1.27)
-				)
-				(hide yes)
-			)
-		)
 		(property "TEST" ""
 			(at 246.38 31.75 0)
@@
 		)
 		(property "MPN" ""
+			(at 246.38 31.75 0)
+			(effects
+				(font
+					(size 1.27 1.27)
+				)
+				(hide yes)
+			)
+		)
+		(property "LCSC" "C13585"
 			(at 246.38 31.75 0)
 			(effects
@@
 			)
 		)
-		(property "LCSC Part #" "C13585"
-			(at 186.69 78.74 0)
-			(effects
-				(font
-					(size 1.27 1.27)
-				)
-				(hide yes)
-			)
-		)
 		(property "TEST" ""
 			(at 186.69 78.74 0)
@@
 			)
 		)
+		(property "LCSC" "C13585"
+			(at 186.69 78.74 0)
+			(effects
+				(font
+					(size 1.27 1.27)
+				)
+				(hide yes)
+			)
+		)
 		(pin "1"
 		)
@@
 			)
 		)
-		(property "LCSC Part #" "C2480"
+		(property "MPN" ""
 			(at 273.05 74.93 0)
 			(effects
@@
 			)
 		)
-		(property "MPN" ""
+		(property "LCSC" "C2480"
 			(at 273.05 74.93 0)
 			(effects
@@
 			)
 		)
-		(property "LCSC Part #" "C32346"
-			(at 53.34 43.18 0)
-			(effects
-				(font
-					(size 1.27 1.27)
-				)
-				(hide yes)
-			)
-		)
 		(property "MPN" ""
+			(at 53.34 43.18 90)
+			(effects
+				(font
+					(size 1.27 1.27)
+				)
+				(hide yes)
+			)
+		)
+		(property "LCSC" "C32346"
 			(at 53.34 43.18 90)
 			(effects
@@
 			)
 		)
-		(property "LCSC Part #" "C2480"
+		(property "MPN" ""
 			(at 241.3 60.96 0)
 			(effects
@@
 			)
 		)
-		(property "MPN" ""
+		(property "LCSC" "C2480"
 			(at 241.3 60.96 0)
 			(effects
@@
 			)
 		)
-		(property "LCSC Part #" "C61063"
-			(at 212.09 77.47 0)
-			(effects
-				(font
-					(size 1.27 1.27)
-				)
-				(hide yes)
-			)
-		)
 		(property "MPN" ""
 			(at 212.09 77.47 0)
 			(effects
+				(font
+					(size 1.27 1.27)
+				)
+				(hide yes)
+			)
+		)
+		(property "LCSC" "C61063"
+			(at 212.09 77.47 0)
+			(effects
